Commit message: Add test_load.py script for loading and controlling mycobot_280m5 robot in PyBullet

File: models/mycobot_280_m5/mycobot_280m5_with_gripper_parallel.urdf (robot description, URDF)
Before this commit: robot firefighter, 15 links, 14 joints
Links:
- link g_base: geometry collision mesh filename=G_base.dae; visual mesh filename=G_base.dae
- link gripper_base: geometry collision mesh filename=gripper_base.dae; visual mesh filename=gripper_base.dae
- link gripper_left1: geometry collision mesh filename=gripper_left1.dae; visual mesh filename=gripper_left1.dae
- link gripper_left2: geometry collision mesh filename=gripper_left2.dae; visual mesh filename=gripper_left2.dae
- link gripper_left3: geometry collision mesh filename=gripper_left3.dae; visual mesh filename=gripper_left3.dae
- link gripper_right1: geometry collision mesh filename=gripper_right1.dae; visual mesh filename=gripper_right1.dae
- link gripper_right2: geometry collision mesh filename=gripper_right2.dae; visual mesh filename=gripper_right2.dae
- link gripper_right3: geometry collision mesh filename=gripper_right3.dae; visual mesh filename=gripper_right3.dae
- link joint1: geometry collision mesh filename=joint1.dae; visual mesh filename=joint1.dae
- link joint2: geometry collision mesh filename=joint2.dae; visual mesh filename=joint2.dae
- link joint3: geometry collision mesh filename=joint3.dae; visual mesh filename=joint3.dae
- link joint4: geometry collision mesh filename=joint4.dae; visual mesh filename=joint4.dae
- link joint5: geometry collision mesh filename=joint5.dae; visual mesh filename=joint5.dae
- link joint6: geometry collision mesh filename=joint6.dae; visual mesh filename=joint6.dae
- link joint6_flange: geometry collision mesh filename=joint7.dae; visual mesh filename=joint7.dae
Joints:
- joint g_base_to_joint1: axis 0 0 0 -> (none); limit lower=-3.14 upper=3.14159 effort=1000.0 velocity=0 -> (none)
- joint joint3_to_joint2: origin xyz=0 0  0 rpy=0 1.5708 -1.5708 -> xyz=0 0 0 rpy=0 1.5708 -1.5708
- joint joint4_to_joint3: axis  0 0 1 -> 0 0 1; origin xyz=  -0.1104 0 0    rpy=0 0 0 -> xyz=-0.1104 0 0 rpy=0 0 0
- joint joint5_to_joint4: axis  0 0 1 -> 0 0 1
